File: cptibp8-pcb/cptibp8-pcb.kicad_pcb (KiCad board)
At the start: 2 copper layers, 51.4 x 43 mm, 51 parts, among them J1 VEXT, J2 OUT, J3 USB_B_Micro, J4 OUT, Q1 AO3401A, Q2 2N7002, U1 MIC2250-1YD5-TR, U2 NCP360SNT, U3 TPS3808DBV, U4 BQ21040, U5 AP63200WU

Commit message: update and plot v0.1
Parts:
- added C13: 1u, Capacitor_SMD:C_0805_2012Metric, B.Cu at (15.8, 17.8)
- added G***: LOGO, LOGO, B.Cu at (46.0, 11.0)
- added J5: VAC1, Connector_PinHeader_2.00mm:PinHeader_1x01_P2.00mm_Vertical, F.Cu at (5.00, 30.7)
- added Q3: DMG2302UK, Package_TO_SOT_SMD:SOT-23, B.Cu at (8.94, 40.1)
- added REF**: graphic_calcpsulogo, george:graphic_calcpsulogo, B.Cu at (47.0, 5.00)
- added REF**: graphic_batterysafety, george:graphic_batterysafety, B.Cu at (34.0, 11.0)
- J1: value VEXT -> VAC2; footprint Connector_PinHeader_2.54mm:PinHeader_1x02_P2.54mm_Horizontal -> Connector_PinHeader_2.00mm:PinHeader_1x01_P2.00mm_Vertical
- J4: footprint Connector_PinHeader_2.54mm:PinHeader_1x03_P2.54mm_Horizontal -> Connector_PinHeader_2.54mm:PinHeader_1x03_P2.54mm_Vertical
- Q2: value 2N7002 -> FDV301N
- moved REF** 10.1 mm to (4.00, 17.0)
- moved C12 3.70 mm to (24.4, 25.9), turned to 180 degrees
- moved D8 3.70 mm to (12.3, 27.6)
- moved J1 3.28 mm to (5.00, 36.8)
- moved C10 0.60 mm to (28.0, 36.7)
- moved C8 0.60 mm to (18.9, 36.7)
- moved BT1 0.57 mm to (42.2, 34.2)
- moved C3 0.50 mm to (21.2, 34.3)
- moved C7 0.50 mm to (27.4, 40.1)
- moved L1 0.50 mm to (22.4, 38.5)
- moved R1 0.50 mm to (21.2, 32.2)
- moved R2 0.50 mm to (24.7, 32.2)
- moved U1 0.50 mm to (27.3, 36.4)
- moved R9 0.49 mm to (48.0, 32.1), turned to 0 degrees
- moved Q2 0.20 mm to (36.3, 25.4)
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- renumbered D4 to locked
Connections:
- J2 pad 1: /GND -> /VOUTN
- J4 pad 1: /GND -> /VOUTN
Routing:
- net /BLOAD: track 41.5 -> 8.05 mm, vias 2 -> 0
- net /EN: track 22.7 -> 45.5 mm
- net /VOUTN: track 0.00 -> 11.5 mm
- net /B+: track 34.3 -> 24.5 mm, vias 1 -> 3
- net /GND: track 6.90 -> 0.00 mm, vias 18 -> 50
- net /VOUT: track 11.4 -> 4.47 mm
- net /RSW: track 10.2 -> 3.67 mm
- net /VINDC: track 23.1 -> 18.3 mm
- net /REG5_SW: track 7.90 -> 3.40 mm
- net /TS: track 27.8 -> 31.7 mm
- net /VCC: track 68.9 -> 65.4 mm
- net /VAC1: track 12.6 -> 9.84 mm
- net /PROG: track 2.72 -> 0.00 mm
- net /VAC2: track 12.9 -> 15.6 mm
- net /PROG2: track 4.51 -> 2.51 mm
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- added copper zone on B.Cu, net /B+
- added copper zone on F.Cu, net /B+
- added copper zone on B.Cu, net /VOUT
Other:
- outline, holes or cut-outs redrawn
- board text added: "+"
- board text added: "CALCPSU"
- board text added: "CHG"
- board text added: "CPTIBP8 V0 7V AC 250mA 5V DC 250mA 9V DC 100mA 3.7V 1600mAh LiPo"
- board text added: "MODEL: SERIAL: INPUT (PINS): INPUT (USB): OUTPUT: BATTERY:"
- board text added: "OUT"
- board text added: "PWR"
- board text added: "github.com/calcpsu/cptibp8"
- board text added: "~IN"
- board text removed: "CALCPSU.COM.AU"
- board text removed: "CPTIBP8 V0 5V DC 400mA 9V DC 100mA 3.7V 2000mAh LiPo"
- board text removed: "MODEL: SERIAL: INPUT: OUTPUT: BATTERY: READ MANUAL BEFORE USING DO NOT SHORT CIRCUIT DO NOT BURN"

Commit message: rev0.3
Parts:
- removed C9: 1u, Capacitor_SMD:C_0805_2012Metric
- removed F2: 0ZCJ0035AF2E, Fuse:Fuse_1210_3225Metric
- removed Q2: FDV301N, Package_TO_SOT_SMD:SOT-23
- removed R13: 33k, Resistor_SMD:R_0805_2012Metric
- removed R15: 4k1, Resistor_SMD:R_0805_2012Metric
- removed R3: 3M3, Resistor_SMD:R_0805_2012Metric
- removed R4: 500k, Resistor_SMD:R_0805_2012Metric
- removed R5: 50k, Resistor_SMD:R_0805_2012Metric
- removed U3: TPS3808DBV, george:SOT-23-6_TI_DBV6
- added R7: 1, Resistor_SMD:R_1210_3225Metric, B.Cu at (14.2, 23.2)
- added TP1: VINDC, TestPoint:TestPoint_Pad_D1.0mm, B.Cu at (21.5, 29.0)
- added TP10: VOUTN, TestPoint:TestPoint_Pad_D1.0mm, B.Cu at (15.4, 40.6)
- added TP2: B+, TestPoint:TestPoint_Pad_D1.0mm, B.Cu at (46.3, 41.9)
- added TP3: BLOAD, TestPoint:TestPoint_Pad_D1.0mm, B.Cu at (33.2, 40.6)
- added TP4: VOUT, TestPoint:TestPoint_Pad_D1.0mm, B.Cu at (18.5, 30.2)
- added TP5: VOUTF, TestPoint:TestPoint_Pad_D1.0mm, B.Cu at (12.5, 30.5)
- added TP6: GND, TestPoint:TestPoint_Pad_D1.0mm, B.Cu at (29.6, 32.0)
- added TP7: EN, TestPoint:TestPoint_Pad_D1.0mm, B.Cu at (35.2, 40.6)
- added TP8: TS, TestPoint:TestPoint_Pad_D1.0mm, B.Cu at (44.0, 33.0)
- added TP9: VCC, TestPoint:TestPoint_Pad_D1.0mm, B.Cu at (31.6, 32.0)
- C2: value 1n -> 1u
- C3: value 4n7 -> 1n
- C4: value 10u -> 22u
- D1: value 1N5817 -> PMEG40T10ERX
- D5, R9: moved to B.Cu
- J3: value USB_B_Micro -> VCC; footprint george:USB_ALIEX_4LEG -> Connector_PinHeader_2.00mm:PinHeader_1x02_P2.00mm_Vertical
- Q1: value AO3401A -> AO3413
- R1: value 93.1k -> 576k
- R14: value 1k3 -> 5k4
- R17: value 50k -> 49.9k
- R2: value 15k -> 91k
- U2: value NCP360SNT -> APX803S-31SA; footprint george:SOT-23-5_TI_DBV5 -> Package_TO_SOT_SMD:SOT-23-3; moved to B.Cu
- moved REF** 36.2 mm to (40.2, 17.7)
- moved R10 19.4 mm to (31.8, 35.0), turned to 0 degrees
- moved Q1 18.8 mm to (31.8, 37.9)
- moved D6 17.7 mm to (35.0, 37.2)
- moved D5 16.0 mm to (19.6, 25.9), turned to 180 degrees
- moved U4 15.7 mm to (38.8, 35.7), turned to 90 degrees
- moved J3 12.5 mm to (48.8, 34.5), turned to 180 degrees
- moved C6 9.91 mm to (43.8, 36.0), turned to 90 degrees
- moved R14 9.42 mm to (36.9, 32.5), turned to 0 degrees
- moved R6 9.09 mm to (38.3, 41.2), turned to 90 degrees
- moved U2 8.81 mm to (41.2, 40.9)
- moved R9 7.37 mm to (41.7, 36.0), turned to -90 degrees
- moved C2 7.37 mm to (40.8, 32.5), turned to 0 degrees
- moved BT1 2.48 mm to (42.1, 36.6), turned to 90 degrees
- moved C5 2.17 mm to (30.8, 16.1), turned to 90 degrees
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Connections:
- C2 pad 1: Net-(U3-SENSE) -> /VCC
- D2 pad 3: Net-(D2-+) -> /VRECT
- D5 pad 1: /VCC -> /REG5_SW
- D5 pad 2: /VBUS -> /GND
- J3 pad 1: /VBUS1 -> /GND
- J3 pad 2: unconnected-(J3-D--Pad2) -> /VCC
- R14 pad 1: /PROG2 -> /GND
- U2 pad 1: /VBUS1 -> /GND
- U2 pad 2: /GND -> /EN
- U2 pad 3: /GND -> /B+
Routing:
- net /VCC: track 65.4 -> 102.1 mm, vias 3 -> 0
- net /CHG: track 0.00 -> 28.8 mm, vias 0 -> 2
- net /TS: track 31.7 -> 10.7 mm
- net /VBUS: track 14.7 -> 0.00 mm, vias 1 -> 0
- net /BLOAD: track 8.05 -> 18.9 mm
- net /VBUS1: track 8.39 -> 0.00 mm
- net Net-(U3-SENSE): track 7.96 -> 0.00 mm
- net /REG5_SW: track 3.40 -> 7.61 mm
- net /EN: track 45.5 -> 41.6 mm, vias 0 -> 2
- net /VOUTN: track 11.5 -> 14.6 mm
- net /VOUT: track 4.47 -> 7.22 mm
- net Net-(D2-+): track 2.56 -> 0.00 mm
- net /PROG2: track 2.51 -> 0.00 mm
- net /VRECT: track 0.00 -> 2.50 mm
- net /RSW: track 3.67 -> 5.95 mm
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- removed copper zone on B.Cu, net /VCC
- removed copper zone on F.Cu, net /VCC
Other:
- outline, holes or cut-outs redrawn
- board text added: "+ -"
- board text added: "+ T -"
- board text added: "BATTERY"

Commit message: rev0 final
Parts:
- removed D5: PMEG40T10ERX, Diode_SMD:D_SOD-123
- moved J5 3.50 mm to (8.00, 32.5)
- moved J1 3.50 mm to (8.00, 35.0)
- moved J2 0.67 mm to (11.1, 32.4)
Routing:
- net /REG5_SW: track 7.61 -> 3.42 mm
- net /VAC1: track 9.84 -> 12.9 mm
- net /VAC2: track 15.6 -> 12.8 mm
- net /VOUTN: track 14.6 -> 14.1 mm
- net /GND: vias 66 -> 59
Changed lines of the file:
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@@
   (net 23 "/VOUTN")
   (footprint "Connector_PinHeader_2.00mm:PinHeader_1x01_P2.00mm_Vertical" (layer "F.Cu")
-    (at 5 36.8 180)
+    (at 8 35 180)
     (descr "Through hole straight pin header, 1x01, 2.00mm pitch, single row")
     (tags "Through hole pin header THT 1x01 2.00mm single row")
@@
   )
   (footprint "Connector_PinHeader_2.00mm:PinHeader_1x02_P2.00mm_Vertical" (layer "F.Cu")
-    (at 10.5 32.1 90)
+    (at 11.1 32.4 90)
     (descr "Through hole straight pin header, 1x02, 2.00mm pitch, single row")
     (tags "Through hole pin header THT 1x02 2.00mm single row")
@@
     (property "ki_keywords" "connector")
     (attr through_hole)
-    (fp_text reference "J2" (at 2.1 -2.3 180) (layer "F.SilkS") hide
+    (fp_text reference "J2" (at 2.1 -2.3) (layer "F.SilkS") hide
         (effects (font (size 1 1) (thickness 0.15)))
     )
@@
   )
   (footprint "Connector_PinHeader_2.00mm:PinHeader_1x01_P2.00mm_Vertical" (layer "F.Cu")
-    (at 5 30.7)
+    (at 8 32.5)
     (descr "Through hole straight pin header, 1x01, 2.00mm pitch, single row")
     (tags "Through hole pin header THT 1x01 2.00mm single row")
@@
       (net 13 "/TS") (pinfunction "1") (pintype "passive"))
   )
-  (footprint "Diode_SMD:D_SOD-123" (layer "B.Cu")
-    (at 19.65 25.9 180)
-    (descr "SOD-123")
-    (tags "SOD-123")
-    (property "Sheetfile" "cptibp8-pcb.kicad_sch")
-    (property "Sheetname" "")
-    (property "ki_description" "40V 1A Schottky Barrier Rectifier Diode, DO-41")
-    (property "ki_keywords" "diode Schottky")
-    (attr smd)
-    (fp_text reference "D5" (at 0 2) (layer "B.SilkS")
-        (effects (font (size 1 1) (thickness 0.15)) (justify mirror))
-    )
-    (fp_text value "PMEG40T10ERX\n" (at 0 -2.1) (layer "B.Fab")
-        (effects (font (size 1 1) (thickness 0.15)) (justify mirror))
-    )
-    (fp_text user "${REFERENCE}" (at 0 2) (layer "B.Fab")
-        (effects (font (size 1 1) (thickness 0.15)) (justify mirror))
-    )
-    (fp_line (start -2.36 -1) (end 1.65 -1)
-      (stroke (width 0.12) (type solid)) (layer "B.SilkS"))
-    (fp_line (start -2.36 1) (end -2.36 -1)
-      (stroke (width 0.12) (type solid)) (layer "B.SilkS"))
-    (fp_line (start -2.36 1) (end 1.65 1)
-      (stroke (width 0.12) (type solid)) (layer "B.SilkS"))
-    (fp_line (start -2.35 1.15) (end -2.35 -1.15)
-      (stroke (width 0.05) (type solid)) (layer "B.CrtYd"))
-    (fp_line (start -2.35 1.15) (end 2.35 1.15)
-      (stroke (width 0.05) (type solid)) (layer "B.CrtYd"))
-    (fp_line (start 2.35 -1.15) (end -2.35 -1.15)
-      (stroke (width 0.05) (type solid)) (layer "B.CrtYd"))
-    (fp_line (start 2.35 1.15) (end 2.35 -1.15)
-      (stroke (width 0.05) (type solid)) (layer "B.CrtYd"))
-    (fp_line (start -1.4 -0.9) (end -1.4 0.9)
-      (stroke (width 0.1) (type solid)) (layer "B.Fab"))
-    (fp_line (start -1.4 0.9) (end 1.4 0.9)
-      (stroke (width 0.1) (type solid)) (layer "B.Fab"))
-    (fp_line (start -0.75 0) (end -0.35 0)
-      (stroke (width 0.1) (type solid)) (layer "B.Fab"))
-    (fp_line (start -0.35 0) (end -0.35 -0.55)
-      (stroke (width 0.1) (type solid)) (layer "B.Fab"))
-    (fp_line (start -0.35 0) (end -0.35 0.55)
-      (stroke (width 0.1) (type solid)) (layer "B.Fab"))
-    (fp_line (start -0.35 0) (end 0.25 0.4)
-      (stroke (width 0.1) (type solid)) (layer "B.Fab"))
-    (fp_line (start 0.25 -0.4) (end -0.35 0)
-      (stroke (width 0.1) (type solid)) (layer "B.Fab"))
-    (fp_line (start 0.25 0) (end 0.75 0)
-      (stroke (width 0.1) (type solid)) (layer "B.Fab"))
-    (fp_line (start 0.25 0.4) (end 0.25 -0.4)
-      (stroke (width 0.1) (type solid)) (layer "B.Fab"))
-    (fp_line (start 1.4 -0.9) (end -1.4 -0.9)
-      (stroke (width 0.1) (type solid)) (layer "B.Fab"))
-    (fp_line (start 1.4 0.9) (end 1.4 -0.9)
-      (stroke (width 0.1) (type solid)) (layer "B.Fab"))
-    (pad "1" smd roundrect (at -1.65 0 180) (size 0.9 1.2) (layers "B.Cu" "B.Paste" "B.Mask") (roundrect_rratio 0.25)
-      (net 15 "/REG5_SW") (pinfunction "K") (pintype "passive"))
-    (pad "2" smd roundrect (at 1.65 0 180) (size 0.9 1.2) (layers "B.Cu" "B.Paste" "B.Mask") (roundrect_rratio 0.25)
-      (net 2 "/GND") (pinfunction "A") (pintype "passive"))
-    (model "${KICAD6_3DMODEL_DIR}/Diode_SMD.3dshapes/D_SOD-123.wrl"
-      (offset (xyz 0 0 0))
-      (scale (xyz 1 1 1))
-      (rotate (xyz 0 0 0))
-    )
-  )
   (footprint "Resistor_SMD:R_0805_2012Metric" (layer "B.Cu")
     (at 49.3 19 90)
@@
     (effects (font (size 1 1) (thickness 0.15)) (justify left bottom))
   )
-  (gr_text "~IN" (at 3.9 29.2) (layer "F.SilkS")
+  (gr_text "~IN" (at 4 30.5) (layer "F.SilkS")
     (effects (font (size 1 1) (thickness 0.15)) (justify left bottom))
   )
-  (gr_text "~IN" (at 3.8 39.4) (layer "F.SilkS")
+  (gr_text "~IN" (at 3.9 37.7) (layer "F.SilkS")
     (effects (font (size 1 1) (thickness 0.15)) (justify left bottom))
   )
@@
   (via (at 37.8 35.7) (size 0.8) (drill 0.4) (layers "F.Cu" "B.Cu") (free) (net 2))
   (via (at 37.5 28.3) (size 0.8) (drill 0.4) (layers "F.Cu" "B.Cu") (free) (net 2))
-  (via (at 6.5 39.2) (size 0.8) (drill 0.4) (layers "F.Cu" "B.Cu") (free) (net 2))
-  (via (at 8.6 30.4) (size 0.8) (drill 0.4) (layers "F.Cu" "B.Cu") (free) (net 2))
-  (via (at 7.5 29) (size 0.8) (drill 0.4) (layers "F.Cu" "B.Cu") (free) (net 2))
-  (via (at 8.9 32.3) (size 0.8) (drill 0.4) (layers "F.Cu" "B.Cu") (free) (net 2))
   (via (at 41 25) (size 0.8) (drill 0.4) (layers "F.Cu" "B.Cu") (free) (net 2))
   (via (at 16.5 25.9) (size 0.8) (drill 0.4) (layers "F.Cu" "B.Cu") (free) (net 2))
@@
   (via (at 28.4 36.4) (size 0.8) (drill 0.4) (layers "F.Cu" "B.Cu") (free) (net 2))
   (via (at 3.9 21.4) (size 0.8) (drill 0.4) (layers "F.Cu" "B.Cu") (free) (net 2))
-  (via (at 8.9 36.2) (size 0.8) (drill 0.4) (layers "F.Cu" "B.Cu") (free) (net 2))
   (via (at 35 25) (size 0.8) (drill 0.4) (layers "F.Cu" "B.Cu") (free) (net 2))
-  (via (at 8.9 34.2) (size 0.8) (drill 0.4) (layers "F.Cu" "B.Cu") (free) (net 2))
   (via (at 19.5 25.9) (size 0.8) (drill 0.4) (layers "F.Cu" "B.Cu") (free) (net 2))
   (via (at 38.8 35.7) (size 0.8) (drill 0.4) (layers "F.Cu" "B.Cu") (free) (net 2))
-  (via (at 8 38) (size 0.8) (drill 0.4) (layers "F.Cu" "B.Cu") (free) (net 2))
   (via (at 7 27) (size 0.8) (drill 0.4) (layers "F.Cu" "B.Cu") (free) (net 2))
   (via (at 22.4 25.9) (size 0.8) (drill 0.4) (layers "F.Cu" "B.Cu") (free) (net 2))
@@
   (segment (start 22.8875 19.8) (end 21.2875 19.8) (width 1) (layer "B.Cu") (net 15))
   (segment (start 23.0875 23.15) (end 21.2875 23.15) (width 0.6) (layer "B.Cu") (net 15))
-  (segment (start 21.3 25.9) (end 21.3 21.7125) (width 0.8) (layer "B.Cu") (net 15))
-  (segment (start 5.5 24.27) (end 5.5 29) (width 0.8) (layer "B.Cu") (net 16))
-  (segment (start 7.7 35.8) (end 6.7 36.8) (width 0.8) (layer "B.Cu") (net 16))
-  (segment (start 6.7 36.8) (end 5 36.8) (width 0.8) (layer "B.Cu") (net 16))
-  (segment (start 5.5 29) (end 7.7 31.2) (width 0.8) (layer "B.Cu") (net 16))
-  (segment (start 7.7 31.2) (end 7.7 35.8) (width 0.8) (layer "B.Cu") (net 16))
-  (segment (start 4.2 23.03) (end 5.5 21.73) (width 0.8) (layer "B.Cu") (net 17))
-  (segment (start 4.2 29.9) (end 4.2 23.03) (width 0.8) (layer "B.Cu") (net 17))
-  (segment (start 5 30.7) (end 4.2 29.9) (width 0.8) (layer "B.Cu") (net 17))
+  (segment (start 5.5 24.27) (end 5.5 27) (width 0.8) (layer "B.Cu") (net 16))
+  (segment (start 9.275 33.725) (end 8 35) (width 0.8) (layer "B.Cu") (net 16))
+  (segment (start 5.5 27) (end 9.275 30.775) (width 0.8) (layer "B.Cu") (net 16))
+  (segment (start 9.275 30.775) (end 9.275 33.725) (width 0.8) (layer "B.Cu") (net 16))
+  (segment (start 4.2 27.2) (end 8 31) (width 0.8) (layer "B.Cu") (net 17))
+  (segment (start 5.5 21.73) (end 4.2 23.03) (width 0.8) (layer "B.Cu") (net 17))
+  (segment (start 4.2 23.03) (end 4.2 27.2) (width 0.8) (layer "B.Cu") (net 17))
+  (segment (start 8 31) (end 8 32.5) (width 0.8) (layer "B.Cu") (net 17))
   (segment (start 11.65 21.73) (end 14.155 21.73) (width 0.6) (layer "B.Cu") (net 18))
   (segment (start 47.2 21.525) (end 47.2 19.875) (width 0.4) (layer "B.Cu") (net 19))
@@
   (segment (start 21.5 29) (end 21.5 27.6) (width 0.25) (layer "B.Cu") (net 20))
   (segment (start 18 27.6) (end 14.2 27.6) (width 0.8) (layer "B.Cu") (net 20))
-  (segment (start 14.2 32.9) (end 13.7 33.4) (width 0.8) (layer "B.Cu") (net 21))
-  (segment (start 15.6 32.9) (end 14.2 32.9) (width 0.8) (layer "B.Cu") (net 21))
-  (segment (start 12.5 30.5) (end 12.5 32.1) (width 0.25) (layer "B.Cu") (net 21))
-  (segment (start 13.7 33.4) (end 12.5 33.4) (width 0.8) (layer "B.Cu") (net 21))
-  (segment (start 12.5 35) (end 12.5 33.4) (width 0.8) (layer "B.Cu") (net 21))
-  (segment (start 12.5 33.4) (end 12.5 32.1) (width 0.8) (layer "B.Cu") (net 21))
-  (segment (start 10.5 38.08) (end 10.5 32.1) (width 0.6) (layer "B.Cu") (net 23))
-  (segment (start 12.5 40.08) (end 10.5 38.08) (width 0.6) (layer "B.Cu") (net 23))
+  (segment (start 12.5 30.5) (end 13.1 31.1) (width 0.25) (layer "B.Cu") (net 21))
+  (segment (start 12.9 32.6) (end 13.1 32.4) (width 0.8) (layer "B.Cu") (net 21))
+  (segment (start 12.9 34.6) (end 12.9 32.6) (width 0.8) (layer "B.Cu") (net 21))
+  (segment (start 13.1 32.4) (end 15.1 32.4) (width 0.8) (layer "B.Cu") (net 21))
+  (segment (start 12.5 35) (end 12.9 34.6) (width 0.8) (layer "B.Cu") (net 21))
+  (segment (start 15.1 32.4) (end 15.6 32.9) (width 0.8) (layer "B.Cu") (net 21))
+  (segment (start 13.1 31.1) (end 13.1 32.4) (width 0.25) (layer "B.Cu") (net 21))
+  (segment (start 11.1 32.4) (end 11.1 38.68) (width 0.6) (layer "B.Cu") (net 23))
   (segment (start 12.5 40.15) (end 12.5 40.08) (width 0.6) (layer "B.Cu") (net 23))
+  (segment (start 11.1 38.68) (end 12.5 40.08) (width 0.6) (layer "B.Cu") (net 23))
   (segment (start 14.88 40.08) (end 15.4 40.6) (width 0.25) (layer "B.Cu") (net 23))
   (segment (start 9.875 40.15) (end 12.5 40.15) (width 0.6) (layer "B.Cu") (net 23))

Commit message: update enclosure and project
Parts:
- added REF**: ENCLOSURE, george:ENCLOSURE, F.Cu at (0.00, 0.00)
Changed lines of the file:
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@@
     )
+  )
+  (footprint "george:ENCLOSURE" (layer "F.Cu")
+    (at 0 0)
+    (attr board_only allow_missing_courtyard)
+    (fp_text reference "REF**" (at 0 -0.5 unlocked) (layer "F.SilkS") hide
+        (effects (font (size 1 1) (thickness 0.15)))
+    )
+    (fp_text value "ENCLOSURE" (at 0 -4 unlocked) (layer "F.Fab")
+        (effects (font (size 1 1) (thickness 0.15)))
+    )
+    (fp_text user "${REFERENCE}" (at 0 4 unlocked) (layer "F.Fab")
+        (effects (font (size 1 1) (thickness 0.15)))
+    )
+    (fp_line (start -3 0) (end 3 0)
+      (stroke (width 0.12) (type default)) (layer "Dwgs.User"))
+    (fp_line (start 0 -3) (end 0 3)
+      (stroke (width 0.12) (type default)) (layer "Dwgs.User"))
+    (fp_circle (center 0 0) (end 0 -2)
+      (stroke (width 0.12) (type default)) (fill none) (layer "Dwgs.User"))
   )
   (footprint "Connector_JST:JST_SH_BM03B-SRSS-TB_1x03-1MP_P1.00mm_Vertical" (layer "F.Cu")

Commit message: rev1
Parts:
- removed C2: 1u, Capacitor_SMD:C_0805_2012Metric
- removed F1: 0ZCJ0035AF2E, Fuse:Fuse_1210_3225Metric
- removed the G*** at (46.0, 11.0)
- removed Q3: DMG2302UK, Package_TO_SOT_SMD:SOT-23
- removed R14: 5k4, Resistor_SMD:R_0805_2012Metric
- removed R6: 1M, Resistor_SMD:R_0805_2012Metric
- removed the REF** at (0.00, 0.00)
- removed the REF** at (47.0, 5.00)
- removed TP10: VOUTN, TestPoint:TestPoint_Pad_D1.0mm
- added C9: 1u, Capacitor_SMD:C_0805_2012Metric, B.Cu at (42.2, 30.8)
- added D5: PMEG40T10ERX, Diode_SMD:D_SOD-123, B.Cu at (46.0, 29.5)
- added G***: LOGO, LOGO, B.Cu at (49.0, 5.00)
- added G***: \, LOGO, B.Cu at (46.0, 11.5)
- added J7: ZX80-B-5P_30_, mod_local:HRS_ZX80-B-5P_30_, F.Cu at (42.6, 38.5)
- added Q2: 2N7002, Package_TO_SOT_SMD:SOT-23, B.Cu at (36.0, 27.2)
- added R12: 3k6, Resistor_SMD:R_0805_2012Metric, B.Cu at (36.0, 24.4)
- added R3: 10k, Resistor_SMD:R_0805_2012Metric, B.Cu at (28.0, 35.0)
- added R4: 10k, Resistor_SMD:R_0805_2012Metric, B.Cu at (48.5, 28.8)
- added R5: 1k8, Resistor_SMD:R_0805_2012Metric, B.Cu at (36.0, 22.4)
- added U3: NCP360SNT, george:SOT-23-5_TI_DBV5, B.Cu at (42.5, 27.8)
- added U6: NCP380, george:SOT-23-5_TI_DBV5, B.Cu at (27.6, 37.9)
- C3: value 1n -> N/P
- R1: value 576k -> 100k
- R2: value 91k -> 16k
- TP5: value VOUTF -> BLOADF
- U2: value APX803S-31SA -> APX809S-31SA
- moved REF** 34.0 mm to (6.25, 17.2)
- moved TP5 17.1 mm to (26.4, 40.6)
- moved U4 16.3 mm to (36.4, 19.6), turned to 180 degrees
- moved C6 15.7 mm to (40.8, 20.6), turned to -90 degrees
- moved R9 15.5 mm to (42.8, 20.6), turned to 90 degrees
- moved TP8 13.4 mm to (45.0, 19.6)
- moved TP2 10.0 mm to (39.0, 35.0)
- moved C4 6.54 mm to (17.1, 30.6), turned to 90 degrees
- moved BT1 6.32 mm to (36.0, 38.3), turned to -90 degrees
- moved TP1 5.58 mm to (26.9, 27.6)
- moved TP4 5.55 mm to (24.1, 30.3)
- moved C7 4.23 mm to (23.1, 40.1)
- moved U1 4.23 mm to (23.1, 36.4)
- moved L1 4.22 mm to (18.2, 38.5)
- moved U2 4.19 mm to (38.4, 37.9), turned to 180 degrees
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Connections:
- C7 pad 1: /BLOAD -> /BLOADF
- J2 pad 1: /VOUTN -> /GND
- J2 pad 2: /VOUTF -> /VOUT
- J4 pad 1: /VOUTN -> /GND
- J4 pad 3: /VOUTF -> /VOUT
- L1 pad 1: /BLOAD -> /BLOADF
- TP5 pad 1: /VOUTF -> /BLOADF
- U1 pad 4: /EN -> /BLOADF
- U1 pad 5: /BLOAD -> /BLOADF
Routing:
- net /EN: track 41.6 -> 20.3 mm, vias 2 -> 0
- net /TS: track 10.7 -> 32.0 mm
- net /VBUS: track 0.00 -> 18.4 mm
- net /BLOADF: track 0.00 -> 16.0 mm
- net /CHG: track 28.8 -> 13.5 mm, vias 2 -> 0
- net /VOUTN: track 14.1 -> 0.00 mm
- net /VCC: track 102.1 -> 88.1 mm
- net /VBUS1: track 0.00 -> 13.9 mm, vias 0 -> 1
- net /B+: track 24.4 -> 36.8 mm, vias 4 -> 2
- net /BLOAD: track 18.9 -> 8.31 mm
- net /VOUT: track 7.22 -> 17.3 mm
- net /VOUTF: track 7.70 -> 0.00 mm
- net /VAC1: track 12.9 -> 5.52 mm
- net /RFB: track 13.8 -> 6.80 mm
- net /VRECT: track 2.50 -> 8.80 mm
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- removed copper zone on B.Cu, net /B+
- removed copper zone on F.Cu, net /B+
- removed copper zone on B.Cu, net /VOUT
Other:
- board text added: "BATT"
- board text added: "BLF"
- board text added: "CPTIBP8 V1 5~9V AC 250mA 5V DC 250mA 9V DC 100mA 3.7V 1600mAh LiPo"
- board text added: "USB"
- board text removed: "BATTERY"
- board text removed: "CPTIBP8 V0 7V AC 250mA 5V DC 250mA 9V DC 100mA 3.7V 1600mAh LiPo"

Commit message: Update kicad file version (8.0)
Parts:
- renumbered locked to D4
