File: cptibp8-pcb/cptibp8-pcb.kicad_sch (KiCad schematic)
At the start: 50 parts, among them J1 VEXT, J2 OUT, J3 USB_B_Micro, J4 OUT, Q1 AO3401A, Q2 2N7002, U1 MIC2250-1YD5-TR, U2 NCP360SNT, U3 TPS3808DBV, U4 BQ21040, U5 AP63200WU

Commit message: update and plot v0.1
Parts:
- removed J1: VEXT, Connector_PinHeader_2.54mm:PinHeader_1x02_P2.54mm_Horizontal, symbol Connector_Generic:Conn_01x02
- added C13: 1u, Capacitor_SMD:C_0805_2012Metric, symbol Device:C
- added J1: VAC2, Connector_PinHeader_2.00mm:PinHeader_1x01_P2.00mm_Vertical, symbol Connector:Conn_01x01_Pin
- added J5: VAC1, Connector_PinHeader_2.00mm:PinHeader_1x01_P2.00mm_Vertical, symbol Connector:Conn_01x01_Pin
- added Q3: DMG2302UK, Package_TO_SOT_SMD:SOT-23, symbol Transistor_FET:2N7002
- J4: footprint Connector_PinHeader_2.54mm:PinHeader_1x03_P2.54mm_Horizontal -> Connector_PinHeader_2.54mm:PinHeader_1x03_P2.54mm_Vertical
- Q2: value 2N7002 -> FDV301N
Connections:
- net EN: now also Q3.1 (G)
- net GND: now also C13.2, Q3.2 (S); no longer J2.1 (Pin_1), J4.1 (Pin_1)
- net VAC1: now also J5.1 (Pin_1)
- net VAC2: now also J1.1 (Pin_1)
- net VCC: now also C13.1
- new net VOUTN: J2.1 (Pin_1), J4.1 (Pin_1), Q3.3 (D)
Other:
- note added: "cin=130pF"
- note added: "tau=130ms"
- moved on the sheet: C5

Commit message: rev0.3
Parts:
- removed C9: 1u, Capacitor_SMD:C_0805_2012Metric, symbol Device:C
- removed F2: 0ZCJ0035AF2E, Fuse:Fuse_1210_3225Metric, symbol Device:Polyfuse
- removed J3: USB_B_Micro, george:USB_ALIEX_4LEG, symbol Connector:USB_B_Micro
- removed Q2: FDV301N, Package_TO_SOT_SMD:SOT-23, symbol Transistor_FET:2N7002
- removed R13: 33k, Resistor_SMD:R_0805_2012Metric, symbol Device:R
- removed R15: 4k1, Resistor_SMD:R_0805_2012Metric, symbol Device:R
- removed R3: 3M3, Resistor_SMD:R_0805_2012Metric, symbol Device:R
- removed R4: 500k, Resistor_SMD:R_0805_2012Metric, symbol Device:R
- removed R5: 50k, Resistor_SMD:R_0805_2012Metric, symbol Device:R
- removed U2: NCP360SNT, george:SOT-23-5_TI_DBV5, symbol kicad_george:NCP360SNT
- removed U3: TPS3808DBV, george:SOT-23-6_TI_DBV6, symbol Power_Supervisor:TPS3808DBV
- added J3: VCC, Connector_PinHeader_2.00mm:PinHeader_1x02_P2.00mm_Vertical, symbol Connector_Generic:Conn_01x02
- added R7: 1, Resistor_SMD:R_1210_3225Metric, symbol Device:R
- added TP1: VINDC, TestPoint:TestPoint_Pad_D1.0mm, symbol Connector:TestPoint
- added TP10: VOUTN, TestPoint:TestPoint_Pad_D1.0mm, symbol Connector:TestPoint
- added TP2: B+, TestPoint:TestPoint_Pad_D1.0mm, symbol Connector:TestPoint
- added TP3: BLOAD, TestPoint:TestPoint_Pad_D1.0mm, symbol Connector:TestPoint
- added TP4: VOUT, TestPoint:TestPoint_Pad_D1.0mm, symbol Connector:TestPoint
- added TP5: VOUTF, TestPoint:TestPoint_Pad_D1.0mm, symbol Connector:TestPoint
- added TP6: GND, TestPoint:TestPoint_Pad_D1.0mm, symbol Connector:TestPoint
- added TP7: EN, TestPoint:TestPoint_Pad_D1.0mm, symbol Connector:TestPoint
- added TP8: TS, TestPoint:TestPoint_Pad_D1.0mm, symbol Connector:TestPoint
- added TP9: VCC, TestPoint:TestPoint_Pad_D1.0mm, symbol Connector:TestPoint
- added U2: APX803S-31SA, Package_TO_SOT_SMD:SOT-23-3, symbol kicad_george:APX803S-XXSA
- C2: value 1n -> 1u
- C3: value 4n7 -> 1n
- C4: value 10u -> 22u
- D1: value 1N5817 -> PMEG40T10ERX
- Q1: value AO3401A -> AO3413
- R1: value 93.1k -> 576k
- R14: value 1k3 -> 5k4
- R2: value 15k -> 91k
- R23: value 50k -> 49.9k
Connections:
- net PROG2 is gone; now on net GND: R14.1
- net VBUS is gone; now on net GND: D5.2 (A)
- net B+: now also TP2.1, U2.3 (VCC)
- net BLOAD: now also TP3.1
- net EN: now also TP7.1, U2.2 (~{RESET})
- net GND: now also J3.1 (Pin_1), TP6.1, U2.1 (GND)
- net REG5_SW: now also D5.1 (K)
- net TS: now also TP8.1
- net VCC: now also C2.1, J3.2 (Pin_2), TP9.1; no longer D5.1 (K)
- net VINDC: now also R7.2, TP1.1
- net VOUT: now also TP4.1
- net VOUTF: now also TP5.1
- net VOUTN: now also TP10.1
- net VRECT: now reaches D2.3 (+)
- net VRECT: now also R7.1
- no-connect marks 6 -> 1
Other:
- note added: "13uA"
- note added: "3.04~3.13V 140~280ms delay"
- note added: "9.0V"
- note added: "Ir=10uA"
- note added: "N.R. FOR AP63200"
- note removed: "10uA"
- note removed: "1uA"
- note removed: "40V 1A Vr ~ 3uA @ 5V/25C Vf 0.4V"
- note removed: "8.9V"
- note removed: "82uA"
- note removed: "<-- 3uA"
- note removed: "RATED: 5.0V/400mA EN38.3 T.7: 10V/800mA"
- note removed: "trip at 3.08V falling, 3.17V rising, +/- 1% 300ms delay"
- company: calcpsu.com.au -> CALCPSU
- moved on the sheet: C3, F1, L1

Commit message: rev0 final
Parts:
- removed D5: PMEG40T10ERX, Diode_SMD:D_SOD-123, symbol Diode:1N5819
Other:
- note removed: "N.R. FOR AP63200"
Changed lines of the file:
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@@
   (title_block
     (title "CALCPACK TI BP8")
-    (date "2024-01-22")
-    (rev "0.3")
+    (date "2024-01-26")
+    (rev "0.4")
     (company "CALCPSU")
     (comment 1 "https://github.com/calcpsu/cptipb8")
@@
   (junction (at 219.075 77.47) (diameter 0) (color 0 0 0 0)
   )
-  (junction (at 137.795 85.09) (diameter 0) (color 0 0 0 0)
-  )
   (junction (at 309.88 115.57) (diameter 0) (color 0 0 0 0)
-  )
-  (junction (at 137.795 115.57) (diameter 0) (color 0 0 0 0)
   )
   (junction (at 83.185 77.47) (diameter 0) (color 0 0 0 0)
@@
     (stroke (width 0) (type default))
   )
-  (wire (pts (xy 137.795 104.14) (xy 137.795 115.57))
-    (stroke (width 0) (type default))
-  )
   (wire (pts (xy 211.455 93.98) (xy 211.455 115.57))
     (stroke (width 0) (type default))
@@
     (stroke (width 0) (type default))
   )
-  (wire (pts (xy 137.795 85.09) (xy 137.795 96.52))
-    (stroke (width 0) (type default))
-  )
   (wire (pts (xy 329.565 113.03) (xy 329.565 115.57))
     (stroke (width 0) (type default))
@@
     (stroke (width 0) (type default))
   )
-  (wire (pts (xy 115.57 115.57) (xy 137.795 115.57))
-    (stroke (width 0) (type default))
-  )
   (wire (pts (xy 107.315 115.57) (xy 115.57 115.57))
     (stroke (width 0) (type default))
@@
     (stroke (width 0) (type default))
   )
-  (wire (pts (xy 137.795 115.57) (xy 149.86 115.57))
+  (wire (pts (xy 115.57 115.57) (xy 149.86 115.57))
     (stroke (width 0) (type default))
   )
@@
     (effects (font (size 1.27 1.27)) (justify left bottom))
   )
-  (text "N.R. FOR AP63200" (at 118.745 104.775 0)
-    (effects (font (size 1.27 1.27)) (justify left bottom))
-  )
   (text "500uA" (at 303.53 104.775 0)
     (effects (font (size 1.27 1.27)) (justify left bottom))
@@
         )
       )
-    )
-  )
-  (symbol (lib_id "Diode:1N5819") (at 137.795 100.33 90) (mirror x) (unit 1)
-    (in_bom yes) (on_board yes) (dnp no)
-    (property "Reference" "D5" (at 134.62 98.7425 90)
-      (effects (font (size 1.27 1.27)) (justify left))
-    )
-    (property "Value" "PMEG40T10ERX\n" (at 134.62 101.2825 90)
-      (effects (font (size 1.27 1.27)) (justify left))
-    )
-    (property "Footprint" "Diode_SMD:D_SOD-123" (at 142.24 100.33 0)
-      (effects (font (size 1.27 1.27)) hide)
-    )
-    (property "Datasheet" "http://www.vishay.com/docs/88525/1n5817.pdf" (at 137.795 100.33 0)
-      (effects (font (size 1.27 1.27)) hide)
-    )
-    (pin "1")
-    (pin "2")
-    (instances
-      (project "cptibp8-pcb"
-        (path "/24b7813b-57c8-4f36-94de-f238a7f97e3d"
-          (reference "D5") (unit 1)
-        )
-      )

Commit message: update enclosure and project
Parts:
- C3: value 1n -> N/P
- R1: value 576k -> 100k
- R10: value 47k -> N/P
- R2: value 91k -> 16k
- R6: value 1M -> N/P
- U2: value APX803S-31SA -> APX809S-31SA
Other:
- note added: "REV1 R6 connect to BLOAD, R1 to 100k, R2 to 16k, C3 nonpop U2 change to APX809S-31SA, R6 nonpop R10 nonpop (not required)"

Commit message: rev1
Parts:
- removed C2: 1u, Capacitor_SMD:C_0805_2012Metric, symbol Device:C
- removed F1: 0ZCJ0035AF2E, Fuse:Fuse_1210_3225Metric, symbol Device:Polyfuse
- removed Q3: DMG2302UK, Package_TO_SOT_SMD:SOT-23, symbol Transistor_FET:2N7002
- removed R14: 5k4, Resistor_SMD:R_0805_2012Metric, symbol Device:R
- removed R6: N/P, Resistor_SMD:R_0805_2012Metric, symbol Device:R
- removed TP10: VOUTN, TestPoint:TestPoint_Pad_D1.0mm, symbol Connector:TestPoint
- added C9: 1u, Capacitor_SMD:C_0805_2012Metric, symbol Device:C
- added D5: PMEG40T10ERX, Diode_SMD:D_SOD-123, symbol Diode:1N5819
- added J7: ZX80-B-5P_30_, mod_local:HRS_ZX80-B-5P_30_, symbol zx80:ZX80-B-5P_30_
- added Q2: 2N7002, Package_TO_SOT_SMD:SOT-23, symbol Transistor_FET:2N7002
- added R12: 3k6, Resistor_SMD:R_0805_2012Metric, symbol Device:R
- added R3, R4: 10k, Resistor_SMD:R_0805_2012Metric, symbol Device:R
- added R5: 1k8, Resistor_SMD:R_0805_2012Metric, symbol Device:R
- added U3: NCP360SNT, george:SOT-23-5_TI_DBV5, symbol kicad_george:NCP360SNT
- added U6: NCP380, george:SOT-23-5_TI_DBV5, symbol Power_Management:AP2171W
- R10: value N/P -> 47k
- TP5: value VOUTF -> BLOADF
Connections:
- net VOUTN is gone; now on net GND: J2.1 (Pin_1), J4.1 (Pin_1)
- net BLOAD: now also U6.5 (IN); no longer C7.1, L1.1, U1.5 (VIN)
- net EN: now also U6.4 (EN); no longer U1.4 (EN)
- net GND: now also C9.2, J7.5 (GND), J7.SH1 (SHIELD), J7.SH2 (SHIELD__1), J7.SH3 (SHIELD__2), J7.SH4 (SHIELD__3), Q2.2 (S), R12.1, R3.1, R4.1, U3.2 (GND), U3.3 (~{EN}), U6.2 (GND)
- net PROG: now also R5.2
- net VCC: now also D5.1 (K)
- net VOUT: now also J2.2 (Pin_2), J4.3 (Pin_3)
- removed net VOUTF: J2.2 (Pin_2), J4.3 (Pin_3), TP5.1
- new net: R3.2, U6.3 (~{FLG})
- new net BLOADF: C7.1, L1.1, TP5.1, U1.4 (EN), U1.5 (VIN), U6.1 (OUT)
- new net PROG2: Q2.3 (D), R12.2, R5.1
- new net VBUS: D5.2 (A), Q2.1 (G), R4.2, U3.5 (OUT)
- new net VBUS1: C9.1, J7.1 (VBUS), U3.1 (IN)
- no-connect marks 1 -> 5
Other:
- note added: "EN38.3 T.7: 10V/800mA"
- note added: "REV1 R6 connect to BLOAD, R1 to 100k, R2 to 16k, C3 n/p U2 change to APX809S-31SA R10, R6 removed Add J7, U3, C9, D5"
- note removed: "REV1 R6 connect to BLOAD, R1 to 100k, R2 to 16k, C3 nonpop U2 change to APX809S-31SA, R6 nonpop R10 nonpop (not required)"
- note removed: "cin=130pF"
- moved on the sheet: BT1, C10, C12, C13, C20, C3, C4, C5, C6, C7, C8, D1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

Commit message: Update kicad file version (8.0)
Parts:
- D6: value PMEG40T10ERX -> PMEG40T10ERX
